Commit message: Debugging RViz visualization

File: gait_analysis_description/urdf/gait_analysis_2880.urdf.xacro (robot description, xacro)
@@ -1,7 +1,9 @@
 <?xml version="1.0" ?>
 <robot name="final" xmlns:xacro="http://www.ros.org/wiki/xacro">
+<!--
 <xacro:include filename="$(find final_description)/urdf/materials.xacro" />
 <xacro:include filename="$(find final_description)/urdf/final.ros2control" />
 <xacro:include filename="$(find final_description)/urdf/final.gazebo" />
+-->
 <link name="base_link">
   <inertial>
@@ -10,16 +12,16 @@
     <inertia ixx="0.003782" iyy="0.013301" izz="0.016842" ixy="0.0" iyz="0.0" ixz="0.0"/>
   </inertial>
-  <visual>
-    <origin xyz="0 0 0" rpy="0 0 0"/>
-    <geometry>
-      <mesh filename="file://$(find final_description)/meshes/base_link.stl"
-            scale="0.001 0.001 0.001"/>
-    </geometry>
-    <material name="silver"/>
-  </visual>
+<visual>
+  <geometry>
+    <box size="1 1 1"/>
+  </geometry>
+  <material name="blue">
+    <color rgba="0 0 1 1"/>
+  </material>
+</visual>
   <collision>
     <origin xyz="0 0 0" rpy="0 0 0"/>
     <geometry>
-      <mesh filename="file://$(find final_description)/meshes/base_link.stl"
+      <mesh filename="package://gait_analysis_description/meshes/base_link.stl"
             scale="0.001 0.001 0.001"/>
     </geometry>
@@ -35,5 +37,5 @@
     <origin xyz="0.064783 3.7e-05 -0.79" rpy="0 0 0"/>
     <geometry>
-      <mesh filename="file://$(find final_description)/meshes/thigh_1.stl"
+      <mesh filename="package://gait_analysis_description/meshes/thigh_1_1.stl"
             scale="0.001 0.001 0.001"/>
     </geometry>
@@ -43,5 +45,5 @@
     <origin xyz="0.064783 3.7e-05 -0.79" rpy="0 0 0"/>
     <geometry>
-      <mesh filename="file://$(find final_description)/meshes/thigh_1.stl"
+      <mesh filename="package://gait_analysis_description/meshes/thigh_1_1.stl"
             scale="0.001 0.001 0.001"/>
     </geometry>
@@ -57,5 +59,5 @@
     <origin xyz="0.064877 -0.000242 -0.41" rpy="0 0 0"/>
     <geometry>
-      <mesh filename="file://$(find final_description)/meshes/shank_1.stl"
+      <mesh filename="package://gait_analysis_description/meshes/shank_1.stl"
             scale="0.001 0.001 0.001"/>
     </geometry>
@@ -65,5 +67,5 @@
     <origin xyz="0.064877 -0.000242 -0.41" rpy="0 0 0"/>
     <geometry>
-      <mesh filename="file://$(find final_description)/meshes/shank_1.stl"
+      <mesh filename="package://gait_analysis_description/meshes/shank_1.stl"
             scale="0.001 0.001 0.001"/>
     </geometry>
@@ -79,5 +81,5 @@
     <origin xyz="0.064989 -2.2e-05 -0.05" rpy="0 0 0"/>
     <geometry>
-      <mesh filename="file://$(find final_description)/meshes/foot_1.stl"
+      <mesh filename="package://gait_analysis_description/meshes/ankle_1.stl"
             scale="0.001 0.001 0.001"/>
     </geometry>
@@ -87,5 +89,5 @@
     <origin xyz="0.064989 -2.2e-05 -0.05" rpy="0 0 0"/>
     <geometry>
-      <mesh filename="file://$(find final_description)/meshes/foot_1.stl"
+      <mesh filename="package://gait_analysis_description/meshes/ankle_1.stl"
             scale="0.001 0.001 0.001"/>
     </geometry>

Commit message: Fix URDF package rename and install missing xacro resources

File: gait_analysis_description/urdf/gait_analysis_2880.urdf.xacro (robot description, xacro)
@@ -1,9 +1,7 @@
 <?xml version="1.0" ?>
 <robot name="final" xmlns:xacro="http://www.ros.org/wiki/xacro">
-<!--
-<xacro:include filename="$(find final_description)/urdf/materials.xacro" />
-<xacro:include filename="$(find final_description)/urdf/final.ros2control" />
-<xacro:include filename="$(find final_description)/urdf/final.gazebo" />
--->
+<xacro:include filename="$(find gait_analysis_description)/urdf/materials.xacro" />
+<xacro:include filename="$(find gait_analysis_description)/urdf/final.ros2control" />
+<xacro:include filename="$(find gait_analysis_description)/urdf/final.gazebo" />
 <link name="base_link">
   <inertial>
@@ -12,17 +10,15 @@
     <inertia ixx="0.003782" iyy="0.013301" izz="0.016842" ixy="0.0" iyz="0.0" ixz="0.0"/>
   </inertial>
-<visual>
-  <geometry>
-    <box size="1 1 1"/>
-  </geometry>
-  <material name="blue">
-    <color rgba="0 0 1 1"/>
-  </material>
-</visual>
+  <visual>
+    <origin xyz="0 0 0" rpy="0 0 0"/>
+    <geometry>
+      <mesh filename="file://$(find gait_analysis_description)/meshes/base_link.stl" scale="0.001 0.001 0.001"/>
+    </geometry>
+    <material name="silver"/>
+  </visual>
   <collision>
     <origin xyz="0 0 0" rpy="0 0 0"/>
     <geometry>
-      <mesh filename="package://gait_analysis_description/meshes/base_link.stl"
-            scale="0.001 0.001 0.001"/>
+      <mesh filename="file://$(find gait_analysis_description)/meshes/base_link.stl" scale="0.001 0.001 0.001"/>
     </geometry>
   </collision>
@@ -37,6 +33,5 @@
     <origin xyz="0.064783 3.7e-05 -0.79" rpy="0 0 0"/>
     <geometry>
-      <mesh filename="package://gait_analysis_description/meshes/thigh_1_1.stl"
-            scale="0.001 0.001 0.001"/>
+      <mesh filename="file://$(find gait_analysis_description)/meshes/thigh_1.stl" scale="0.001 0.001 0.001"/>
     </geometry>
     <material name="silver"/>
@@ -45,6 +40,5 @@
     <origin xyz="0.064783 3.7e-05 -0.79" rpy="0 0 0"/>
     <geometry>
-      <mesh filename="package://gait_analysis_description/meshes/thigh_1_1.stl"
-            scale="0.001 0.001 0.001"/>
+      <mesh filename="file://$(find gait_analysis_description)/meshes/thigh_1.stl" scale="0.001 0.001 0.001"/>
     </geometry>
   </collision>
@@ -59,6 +53,5 @@
     <origin xyz="0.064877 -0.000242 -0.41" rpy="0 0 0"/>
     <geometry>
-      <mesh filename="package://gait_analysis_description/meshes/shank_1.stl"
-            scale="0.001 0.001 0.001"/>
+      <mesh filename="file://$(find gait_analysis_description)/meshes/shank_1.stl" scale="0.001 0.001 0.001"/>
     </geometry>
     <material name="silver"/>
@@ -67,6 +60,5 @@
     <origin xyz="0.064877 -0.000242 -0.41" rpy="0 0 0"/>
     <geometry>
-      <mesh filename="package://gait_analysis_description/meshes/shank_1.stl"
-            scale="0.001 0.001 0.001"/>
+      <mesh filename="file://$(find gait_analysis_description)/meshes/shank_1.stl" scale="0.001 0.001 0.001"/>
     </geometry>
   </collision>
@@ -81,6 +73,5 @@
     <origin xyz="0.064989 -2.2e-05 -0.05" rpy="0 0 0"/>
     <geometry>
-      <mesh filename="package://gait_analysis_description/meshes/ankle_1.stl"
-            scale="0.001 0.001 0.001"/>
+      <mesh filename="file://$(find gait_analysis_description)/meshes/foot_1.stl" scale="0.001 0.001 0.001"/>
     </geometry>
     <material name="silver"/>
@@ -89,6 +80,5 @@
     <origin xyz="0.064989 -2.2e-05 -0.05" rpy="0 0 0"/>
     <geometry>
-      <mesh filename="package://gait_analysis_description/meshes/ankle_1.stl"
-            scale="0.001 0.001 0.001"/>
+      <mesh filename="file://$(find gait_analysis_description)/meshes/foot_1.stl" scale="0.001 0.001 0.001"/>
     </geometry>
   </collision>

Commit message: gait_analysis updated

File: gait_analysis_description/urdf/gait_analysis_2880.urdf.xacro (robot description, xacro)
@@ -1,7 +1,7 @@
 <?xml version="1.0" ?>
-<robot name="final" xmlns:xacro="http://www.ros.org/wiki/xacro">
-<xacro:include filename="$(find final_description)/urdf/materials.xacro" />
-<xacro:include filename="$(find final_description)/urdf/final.ros2control" />
-<xacro:include filename="$(find final_description)/urdf/final.gazebo" />
+<robot name="gait_analysis" xmlns:xacro="http://www.ros.org/wiki/xacro">
+<xacro:include filename="$(find gait_analysis_description)/urdf/materials.xacro" />
+<xacro:include filename="$(find gait_analysis_description)/urdf/gait_analysis.ros2control" />
+<xacro:include filename="$(find gait_analysis_description)/urdf/gait_analysis.gazebo" />
 <link name="base_link">
   <inertial>
@@ -13,6 +13,5 @@
     <origin xyz="0 0 0" rpy="0 0 0"/>
     <geometry>
-      <mesh filename="file://$(find final_description)/meshes/base_link.stl"
-            scale="0.001 0.001 0.001"/>
+      <mesh filename="file://$(find gait_analysis_description)/meshes/base_link.stl" scale="0.001 0.001 0.001"/>
     </geometry>
     <material name="silver"/>
@@ -21,6 +20,5 @@
     <origin xyz="0 0 0" rpy="0 0 0"/>
     <geometry>
-      <mesh filename="file://$(find final_description)/meshes/base_link.stl"
-            scale="0.001 0.001 0.001"/>
+      <mesh filename="file://$(find gait_analysis_description)/meshes/base_link.stl" scale="0.001 0.001 0.001"/>
     </geometry>
   </collision>
@@ -35,6 +33,5 @@
     <origin xyz="0.064783 3.7e-05 -0.79" rpy="0 0 0"/>
     <geometry>
-      <mesh filename="file://$(find final_description)/meshes/thigh_1.stl"
-            scale="0.001 0.001 0.001"/>
+      <mesh filename="file://$(find gait_analysis_description)/meshes/thigh_1.stl" scale="0.001 0.001 0.001"/>
     </geometry>
     <material name="silver"/>
@@ -43,6 +40,5 @@
     <origin xyz="0.064783 3.7e-05 -0.79" rpy="0 0 0"/>
     <geometry>
-      <mesh filename="file://$(find final_description)/meshes/thigh_1.stl"
-            scale="0.001 0.001 0.001"/>
+      <mesh filename="file://$(find gait_analysis_description)/meshes/thigh_1.stl" scale="0.001 0.001 0.001"/>
     </geometry>
   </collision>
@@ -57,6 +53,5 @@
     <origin xyz="0.064877 -0.000242 -0.41" rpy="0 0 0"/>
     <geometry>
-      <mesh filename="file://$(find final_description)/meshes/shank_1.stl"
-            scale="0.001 0.001 0.001"/>
+      <mesh filename="file://$(find gait_analysis_description)/meshes/shank_1.stl" scale="0.001 0.001 0.001"/>
     </geometry>
     <material name="silver"/>
@@ -65,6 +60,5 @@
     <origin xyz="0.064877 -0.000242 -0.41" rpy="0 0 0"/>
     <geometry>
-      <mesh filename="file://$(find final_description)/meshes/shank_1.stl"
-            scale="0.001 0.001 0.001"/>
+      <mesh filename="file://$(find gait_analysis_description)/meshes/shank_1.stl" scale="0.001 0.001 0.001"/>
     </geometry>
   </collision>
@@ -79,6 +73,5 @@
     <origin xyz="0.064989 -2.2e-05 -0.05" rpy="0 0 0"/>
     <geometry>
-      <mesh filename="file://$(find final_description)/meshes/foot_1.stl"
-            scale="0.001 0.001 0.001"/>
+      <mesh filename="file://$(find gait_analysis_description)/meshes/foot_1.stl" scale="0.001 0.001 0.001"/>
     </geometry>
     <material name="silver"/>
@@ -87,6 +80,5 @@
     <origin xyz="0.064989 -2.2e-05 -0.05" rpy="0 0 0"/>
     <geometry>
-      <mesh filename="file://$(find final_description)/meshes/foot_1.stl"
-            scale="0.001 0.001 0.001"/>
+      <mesh filename="file://$(find gait_analysis_description)/meshes/foot_1.stl" scale="0.001 0.001 0.001"/>
     </geometry>
   </collision>
